File: kicad/waterLevelMeasurementRabben.kicad_sch (KiCad schematic)
At the start: 3 parts, among them J1 Screw_Terminal_01x02, U1 LM7805_TO220

Commit message: Initial commit
Connections:
- net Earth: now reaches A1.29 (GND)
- net Earth: now also A1.6 (GND), A1.7 (GND), J1.1 (Pin_1), U1.2 (GND)
- net at A1.5 (+5V): now also U1.3 (VO)
- net at J1.2 (Pin_2): now also U1.1 (VI)
Other:
- note added: "1"
- moved on the sheet: A1, J1, U1

Commit message: Initial commit
Parts:
- removed J1: Screw_Terminal_01x02, symbol Connector:Screw_Terminal_01x02
- added J1, J4: OSTTC022162, digikey-footprints:Term_Block_1x2_P5.08MM, symbol dk_Terminal-Blocks-Wire-to-Board:OSTTC022162
- added J2: 0022232031, digikey-footprints:PinHeader_1x3_P2.54mm_Drill1.02mm, symbol dk_Rectangular-Connectors-Headers-Male-Pins:0022232031
Connections:
- net Earth: now also J1.2
- net at U1.1 (VI): now also J1.1
